Commit message: add lidar, cameras, ros2_control

File: description/main_robot.xacro (robot description, xacro)
@@ -5,7 +5,5 @@
     <xacro:property name="chassis_width" value="0.4" />
     <xacro:property name="chassis_height" value="0.1" />
-    <!-- CHANGE THIS -->
     <xacro:property name="chassis_mass" value="1" />
-    <xacro:property name="arm_mass" value="0.001" />
     <xacro:property name="wheel_length" value="0.02" />
     <xacro:property name="wheel_radius" value="0.05" />

File: description/robot.urdf.xacro (robot description, xacro)
@@ -2,3 +2,18 @@
 <robot xmlns:xacro="http://www.ros.org/wiki/xacro"  name="robot">
     <xacro:include filename="main_robot.xacro" />
+    <xacro:include filename="lidar.xacro" />
+    <xacro:arg name="use_depth_cam" default="true"/>
+    <xacro:if value="$(arg use_depth_cam)">
+        <xacro:include filename="depth_camera.xacro"/>
+    </xacro:if>
+    <xacro:unless value="$(arg use_depth_cam)">
+        <xacro:include filename="camera.xacro"/>
+    </xacro:unless>
+    <xacro:arg name="use_ros2_control" default="true"/>
+    <xacro:if value="$(arg use_ros2_control)">
+        <xacro:include filename="gazebo_ros2_control.xacro" />
+    </xacro:if>
+    <xacro:unless value="$(arg use_ros2_control)">
+        <xacro:include filename="gazebo_diff_drive.xacro" />
+    </xacro:unless>
 </robot>
