Commit message: add robot_localization node, rtabmap

File: description/depth_camera.xacro (robot description, xacro)
@@ -1,10 +1,22 @@
 <?xml version="1.0"?>
 <robot xmlns:xacro="http://www.ros.org/wiki/xacro">
-    <joint name="depth_camera_joint" type="fixed">
+    <joint name="camera_joint" type="fixed">
         <parent link="chassis_link"/>
-        <child link="depth_camera_link"/>
+        <child link="camera_link"/>
         <origin xyz="0.35 0 0.14" rpy="0 0 0"/>
     </joint>
-    <link name="depth_camera_link">
+    <joint name="camera_rgb_joint" type="fixed">
+        <parent link="camera_link"/>
+        <child link="camera_rgb_frame"/>
+        <origin xyz="0 0 0" rpy="0 0 0"/>
+    </joint>
+    <joint name="camera_rgb_optical_joint" type="fixed">
+        <parent link="camera_rgb_frame"/>
+        <child link="camera_rgb_optical_frame"/>
+        <origin xyz="0 0 0" rpy="${-pi/2} 0 ${-pi/2}"/>
+    </joint>
+    <link name="camera_link"/>
+    <link name="camera_rgb_optical_frame"/>
+    <link name="camera_rgb_frame">
         <visual>
             <geometry>
@@ -21,16 +33,11 @@
         </visual>
     </link>
-        <joint name="depth_camera_optical_joint" type="fixed">
-        <parent link="depth_camera_link"/>
-        <child link="depth_camera_link_optical"/>
-        <origin xyz="0 0 0" rpy="${-pi/2} 0 ${-pi/2}"/>
-    </joint>
-    <link name="depth_camera_link_optical"></link>
-    <gazebo reference="depth_camera_link">
+    <!-- <link name="depth_camera_link_optical"></link> -->
+    <gazebo reference="camera_rgb_frame">
         <material>Gazebo/Black</material>
-        <sensor name="depth_camera" type="depth">
+        <sensor name="camera" type="depth">
             <pose> 0 0 0 0 0 0 </pose>
             <visualize>true</visualize>
-            <update_rate>10</update_rate>
+            <update_rate>30</update_rate>
             <camera>
                 <horizontal_fov>1.089</horizontal_fov>
@@ -42,10 +49,10 @@
                 <clip>
                     <near>0.05</near>
-                    <far>8.0</far>
+                    <far>300.0</far>
                 </clip>
             </camera>
             <plugin name="camera_controller" filename="libgazebo_ros_camera.so">
-                <frame_name>depth_camera_link_optical</frame_name>
-                <min_depth>0.1</min_depth>
+                <frame_name>camera_rgb_optical_frame</frame_name>
+                <min_depth>0.3</min_depth>
                 <max_depth>100.0</max_depth>
             </plugin>

File: description/gazebo_ros2_control.xacro (robot description, xacro)
@@ -24,5 +24,5 @@
     <gazebo>
         <plugin filename="libgazebo_ros2_control.so" name="gazebo_ros2_control">
-            <parameters>$(find diffbot_scara)/config/my_controllers.yaml</parameters>
+            <parameters>$(find diffbot_gazebo)/config/my_controllers.yaml</parameters>
         </plugin>
     </gazebo>

File: description/robot.urdf.xacro (robot description, xacro)
@@ -3,4 +3,5 @@
     <xacro:include filename="main_robot.xacro" />
     <xacro:include filename="lidar.xacro" />
+    <xacro:include filename="imu.xacro" />
     <xacro:arg name="use_depth_cam" default="true"/>
     <xacro:if value="$(arg use_depth_cam)">
