Commit message: doing visual odometry

File: description/camera.xacro (robot description, xacro)
@@ -2,5 +2,5 @@
 <robot xmlns:xacro="http://www.ros.org/wiki/xacro">
     <joint name="camera_joint" type="fixed">
-        <parent link="chassis_link"/>
+        <parent link="base_link"/>
         <child link="camera_link"/>
         <origin xyz="0.35 0 0.14" rpy="0 0 0"/>

File: description/main_robot.xacro (robot description, xacro)
@@ -32,4 +32,5 @@
             <geometry>
                 <box size= "${chassis_length} ${chassis_width} ${chassis_height}"/>
+                <!-- <mesh filename="package://diffbot_gazebo/description/Omni_3_Bot.dae" scale="1 1 1" /> -->
             </geometry>
             <material name="red"/>
